File: assets/kicad/ADBv2.kicad_pcb (KiCad board)
At the start: 2 copper layers, 126.6 x 21.4 mm, 17 parts, among them J2 TOP, J3 BOTTOM, J4 BAT, SW1 MINI MSK12CO2, U1 MCP23017-E/SS, U2 MCP23017-E/SS

Commit message: changes to zmk files
Other:
- board text added: "ljwilliams"
- board text removed: "ADBv2 https://mtt.cx"
