File: assets/kicad/ADBv2.kicad_sch (KiCad schematic)
At the start: 17 parts, among them J1 EC11, J2 TOP, J3 BOTTOM, J4 BAT, J5 SPI, SW1 MINI MSK12CO2, U1 MCP23017-E/SS, U2 MCP23017-E/SS

Commit message: changes to zmk files
Other:
- company: mtt.cx -> ljwilliams09
Changed lines of the file:
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@@
 (kicad_sch
-	(version 20231120)
+	(version 20250114)
 	(generator "eeschema")
-	(generator_version "8.0")
+	(generator_version "9.0")
 	(paper "A4")
 	(title_block
 		(title "ADB")
 		(rev "2")
-		(company "mtt.cx")
+		(company "ljwilliams09")
 	)
 	(junction
@@
 		)
 	)
+	(embedded_fonts no)
 )
